File: kicad/eink_badge.kicad_pcb (KiCad board)
At the start: 2 copper layers, 77.5 x 42.5 mm, 78 parts, among them CN2 B2B-PH-K-S, Q1 AO3400A, SW1 MST-12D18G2 SMD SLIDE SWITCH, U1 RP2350A, U10 TPS63060DSCR, U2 NCP1117-3.3_SOT223, U3 GT-USB-7010ASV, U4 W25Q128JVS, U5 YZA-009, U6 ABM8-272-T3_C20625731, U7 SM03B-SRSS-TB, U8 CY43-10UH, U9 BQ24040DSQR

Commit message: Refactor code structure for improved readability and maintainability
Other:
- board size 77.5 x 42.5 mm -> 77.5 x 48.5 mm
