File: kicad/battery_charger.kicad_sch (KiCad schematic)
At the start: 19 parts, among them CN2 B2B-PH-K-S, U10 TPS63060DSCR, U9 BQ24040DSQR

Commit message: Changed to use foorprint of 0603 0805 1005 metric for resistors and capacitors where possible
Parts:
- C23: footprint easyeda2kicad:C0805 -> Capacitor_SMD:C_0805_2012Metric
- C24, C30, C35: value LMK212BJ226MG-T -> 22uF; footprint easyeda2kicad:C0805 -> Capacitor_SMD:C_0805_2012Metric
- C28, C36: value EMK212BJ106KG-T -> 10uF; footprint easyeda2kicad:C0805 -> Capacitor_SMD:C_0805_2012Metric
- C37: value CC0402KRX5R9BB104 -> 0.1uF; footprint easyeda2kicad:C0402 -> Capacitor_SMD:C_0603_1608Metric; LCSC Part C105882 -> (none); MPN CC0402KRX5R9BB104 -> (none); Manufacturer YAGEO(国巨) -> (none)
- C38: value CL10C100JB8NNNC -> 10pF; footprint easyeda2kicad:C0603 -> Capacitor_SMD:C_0603_1608Metric
- R12, R8: footprint Resistor_SMD:R_0402_1005Metric -> Resistor_SMD:R_0603_1608Metric
- R20: footprint Resistor_SMD:R_0201_0603Metric -> Resistor_SMD:R_0603_1608Metric
Changed lines of the file:
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@@
 			)
 		)
-		(property "Footprint" "Resistor_SMD:R_0201_0603Metric"
+		(property "Footprint" "Resistor_SMD:R_0603_1608Metric"
 			(at 155.702 143.51 90)
 			(hide yes)
@@
 			)
 		)
-		(property "Value" "CL10C100JB8NNNC"
+		(property "Value" "10pF"
 			(at 180.34 144.7799 90)
 			(hide yes)
@@
 			)
 		)
-		(property "Footprint" "easyeda2kicad:C0603"
+		(property "Footprint" "Capacitor_SMD:C_0603_1608Metric"
 			(at 184.15 143.51 0)
 			(hide yes)
@@
 			)
 		)
-		(property "Footprint" "easyeda2kicad:C0805"
+		(property "Footprint" "Capacitor_SMD:C_0805_2012Metric"
 			(at 114.3 80.01 0)
 			(hide yes)
@@
 			)
 		)
-		(property "Datasheet" "https://lcsc.com/product-detail/Multilayer-Ceramic-Capacitors-MLCC-SMD-SMT_SAMSUNG_CL21A475KAQNNNE_4-7uF-475-10-25V_C1779.html"
+		(property "Datasheet" ""
 			(at 116.84 80.01 0)
 			(hide yes)
@@
 			)
 		)
-		(property "Value" "CC0402KRX5R9BB104"
+		(property "Value" "0.1uF"
 			(at 148.59 140.97 0)
 			(hide yes)
@@
 			)
 		)
-		(property "Footprint" "easyeda2kicad:C0402"
+		(property "Footprint" "Capacitor_SMD:C_0603_1608Metric"
 			(at 160.02 140.97 0)
 			(hide yes)
@@
 			)
 		)
-		(property "Datasheet" "https://lcsc.com/product-detail/Multilayer-Ceramic-Capacitors-MLCC-SMD-SMT_100nF-104-10-50V_C105882.html"
+		(property "Datasheet" ""
 			(at 162.56 140.97 0)
 			(hide yes)
@@
 			)
 		)
-		(property "Manufacturer" "YAGEO(国巨)"
+		(property "Manufacturer" ""
 			(at 165.1 140.97 0)
 			(hide yes)
@@
 			)
 		)
-		(property "MPN" "CC0402KRX5R9BB104"
+		(property "MPN" ""
 			(at 167.64 140.97 0)
 			(hide yes)
@@
 			)
 		)
-		(property "LCSC Part" "C105882"
+		(property "LCSC Part" ""
 			(at 170.18 140.97 0)
 			(hide yes)
@@
 			)
 		)
-		(property "Footprint" "Resistor_SMD:R_0402_1005Metric"
+		(property "Footprint" "Resistor_SMD:R_0603_1608Metric"
 			(at 38.862 88.9 90)
 			(hide yes)
@@
 			)
 		)
-		(property "Value" "LMK212BJ226MG-T"
+		(property "Value" "22uF"
 			(at 200.66 134.62 0)
 			(hide yes)
@@
 			)
 		)
-		(property "Footprint" "easyeda2kicad:C0805"
+		(property "Footprint" "Capacitor_SMD:C_0805_2012Metric"
 			(at 189.23 134.62 0)
 			(hide yes)
@@
 			)
 		)
-		(property "Datasheet" "https://lcsc.com/product-detail/Multilayer-Ceramic-Capacitors-MLCC-SMD-SMT_TAIYO-YUDEN_LMK212BJ226MG-T_22uF-226-20-10V_C92814.html"
+		(property "Datasheet" ""
 			(at 186.69 134.62 0)
 			(hide yes)
@@
 			)
 		)
-		(property "Footprint" "Resistor_SMD:R_0402_1005Metric"
+		(property "Footprint" "Resistor_SMD:R_0603_1608Metric"
 			(at 27.432 88.9 90)
 			(hide yes)
@@
 			)
 		)
-		(property "Value" "LMK212BJ226MG-T"
+		(property "Value" "22uF"
 			(at 196.85 134.62 0)
 			(hide yes)
@@
 			)
 		)
-		(property "Footprint" "easyeda2kicad:C0805"
+		(property "Footprint" "Capacitor_SMD:C_0805_2012Metric"
 			(at 185.42 134.62 0)
 			(hide yes)
@@
 			)
 		)
-		(property "Datasheet" "https://lcsc.com/product-detail/Multilayer-Ceramic-Capacitors-MLCC-SMD-SMT_TAIYO-YUDEN_LMK212BJ226MG-T_22uF-226-20-10V_C92814.html"
+		(property "Datasheet" ""
 			(at 182.88 134.62 0)
 			(hide yes)
@@
 			)
 		)
-		(property "Value" "EMK212BJ106KG-T"
+		(property "Value" "10uF"
 			(at 101.6 134.6199 90)
 			(hide yes)
@@
 			)
 		)
-		(property "Footprint" "easyeda2kicad:C0805"
+		(property "Footprint" "Capacitor_SMD:C_0805_2012Metric"
 			(at 105.41 133.35 0)
 			(hide yes)
@@
 			)
 		)
-		(property "Datasheet" "https://lcsc.com/product-detail/Multilayer-Ceramic-Capacitors-MLCC-SMD-SMT_TAIYO-YUDEN_EMK212BJ106KG-T_10uF-106-10-16V_C87157.html"
+		(property "Datasheet" ""
 			(at 107.95 133.35 0)
 			(hide yes)
@@
 			)
 		)
-		(property "Value" "LMK212BJ226MG-T"
+		(property "Value" "22uF"
 			(at 204.47 134.62 0)
 			(hide yes)
@@
 			)
 		)
-		(property "Footprint" "easyeda2kicad:C0805"
+		(property "Footprint" "Capacitor_SMD:C_0805_2012Metric"
 			(at 193.04 134.62 0)
 			(hide yes)
@@
 			)
 		)
-		(property "Datasheet" "https://lcsc.com/product-detail/Multilayer-Ceramic-Capacitors-MLCC-SMD-SMT_TAIYO-YUDEN_LMK212BJ226MG-T_22uF-226-20-10V_C92814.html"
+		(property "Datasheet" ""
 			(at 190.5 134.62 0)
 			(hide yes)
@@
 			)
 		)
-		(property "Value" "EMK212BJ106KG-T"
+		(property "Value" "10uF"
 			(at 96.52 134.6199 90)
 			(hide yes)
@@
 			)
 		)
-		(property "Footprint" "easyeda2kicad:C0805"
+		(property "Footprint" "Capacitor_SMD:C_0805_2012Metric"
 			(at 100.33 133.35 0)
 			(hide yes)
@@
 			)
 		)
-		(property "Datasheet" "https://lcsc.com/product-detail/Multilayer-Ceramic-Capacitors-MLCC-SMD-SMT_TAIYO-YUDEN_EMK212BJ106KG-T_10uF-106-10-16V_C87157.html"
+		(property "Datasheet" ""
 			(at 102.87 133.35 0)
 			(hide yes)
