File: kicad/untitled.kicad_sch (KiCad schematic)
At the start: 25 parts, among them Q1 AO3400A, SW1 MST-12D18G2 SMD SLIDE SWITCH, U8 CY43-10UH

Commit message: Changed to use foorprint of 0603 0805 1005 metric for resistors and capacitors where possible
Parts:
- C19, C20, C21, C22, C25, C26, C27, C29: footprint easyeda2kicad:C0805 -> Capacitor_SMD:C_0805_2012Metric
- C31, C32, C33, C34: value CL10A105KB8NNNC -> 1uF; footprint easyeda2kicad:C0603 -> Capacitor_SMD:C_0603_1608Metric
- R10, R11: value 0603WAF220KT5E -> 2.2; footprint easyeda2kicad:R0603 -> Resistor_SMD:R_0603_1608Metric
- R13: value 0402WGF1002TCE -> 10k; footprint easyeda2kicad:R0402 -> Resistor_SMD:R_0603_1608Metric; LCSC Part C25744 -> C115324; MPN 0402WGF1002TCE -> (none); Manufacturer UNI-ROYAL(厚声) -> (none)
- R14: value 0402WGF1002TCE -> 10k
- R15, R16: value 0603WAF100KT5E -> 1
Changed lines of the file:
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@@
 			)
 		)
-		(property "Value" "0603WAF100KT5E"
+		(property "Value" "1"
 			(at 91.44 109.2199 90)
 			(hide yes)
@@
 			)
 		)
-		(property "Datasheet" "https://lcsc.com/product-detail/Chip-Resistor-Surface-Mount-UniOhm_1R-1R00-1_C22936.html"
+		(property "Datasheet" ""
 			(at 99.06 107.95 0)
 			(hide yes)
@@
 			)
 		)
-		(property "Value" "0603WAF220KT5E"
+		(property "Value" "2.2"
 			(at 68.58 107.9499 90)
 			(hide yes)
@@
 			)
 		)
-		(property "Footprint" "easyeda2kicad:R0603"
+		(property "Footprint" "Resistor_SMD:R_0603_1608Metric"
 			(at 73.66 106.68 0)
 			(hide yes)
@@
 			)
 		)
-		(property "Datasheet" "https://lcsc.com/product-detail/Chip-Resistor-Surface-Mount-UniOhm_2-2R-2R20-1_C22939.html"
+		(property "Datasheet" ""
 			(at 76.2 106.68 0)
 			(hide yes)
@@
 			)
 		)
-		(property "Value" "0402WGF1002TCE"
+		(property "Value" "10k"
 			(at 57.15 96.5199 90)
 			(hide yes)
@@
 			)
 		)
-		(property "Footprint" "easyeda2kicad:R0402"
+		(property "Footprint" "Resistor_SMD:R_0603_1608Metric"
 			(at 62.23 95.25 0)
 			(hide yes)
@@
 			)
 		)
-		(property "Datasheet" "https://lcsc.com/product-detail/Chip-Resistor-Surface-Mount-UniOhm_10KR-1002-1_C25744.html"
+		(property "Datasheet" ""
 			(at 64.77 95.25 0)
 			(hide yes)
@@
 			)
 		)
-		(property "Manufacturer" "UNI-ROYAL(厚声)"
+		(property "Manufacturer" ""
 			(at 67.31 95.25 0)
 			(hide yes)
@@
 			)
 		)
-		(property "MPN" "0402WGF1002TCE"
+		(property "MPN" ""
 			(at 69.85 95.25 0)
 			(hide yes)
@@
 			)
 		)
-		(property "LCSC Part" "C25744"
+		(property "LCSC Part" "C115324"
 			(at 72.39 95.25 0)
 			(hide yes)
@@
 			)
 		)
-		(property "Footprint" "easyeda2kicad:C0805"
+		(property "Footprint" "Capacitor_SMD:C_0805_2012Metric"
 			(at 73.66 60.96 0)
 			(hide yes)
@@
 			)
 		)
-		(property "Datasheet" "https://lcsc.com/product-detail/Multilayer-Ceramic-Capacitors-MLCC-SMD-SMT_SAMSUNG_CL21A475KAQNNNE_4-7uF-475-10-25V_C1779.html"
+		(property "Datasheet" ""
 			(at 76.2 60.96 0)
 			(hide yes)
@@
 			)
 		)
-		(property "Footprint" "easyeda2kicad:C0805"
+		(property "Footprint" "Capacitor_SMD:C_0805_2012Metric"
 			(at 106.68 116.84 0)
 			(hide yes)
@@
 			)
 		)
-		(property "Datasheet" "https://lcsc.com/product-detail/Multilayer-Ceramic-Capacitors-MLCC-SMD-SMT_SAMSUNG_CL21A475KAQNNNE_4-7uF-475-10-25V_C1779.html"
+		(property "Datasheet" ""
 			(at 106.68 119.38 0)
 			(hide yes)
@@
 		(dnp no)
 		(property "Reference" "C22"
-			(at 115.316 74.422 0)
+			(at 112.776 72.898 0)
 			(show_name no)
 			(do_not_autoplace no)
@@
 			)
 		)
-		(property "Footprint" "easyeda2kicad:C0805"
+		(property "Footprint" "Capacitor_SMD:C_0805_2012Metric"
 			(at 115.57 63.5 0)
 			(hide yes)
@@
 			)
 		)
-		(property "Datasheet" "https://lcsc.com/product-detail/Multilayer-Ceramic-Capacitors-MLCC-SMD-SMT_SAMSUNG_CL21A475KAQNNNE_4-7uF-475-10-25V_C1779.html"
+		(property "Datasheet" ""
 			(at 115.57 60.96 0)
 			(hide yes)
@@
 			)
 		)
-		(property "Footprint" "easyeda2kicad:C0805"
+		(property "Footprint" "Capacitor_SMD:C_0805_2012Metric"
 			(at 105.41 124.46 0)
 			(hide yes)
@@
 			)
 		)
-		(property "Datasheet" "https://lcsc.com/product-detail/Multilayer-Ceramic-Capacitors-MLCC-SMD-SMT_SAMSUNG_CL21A475KAQNNNE_4-7uF-475-10-25V_C1779.html"
+		(property "Datasheet" ""
 			(at 105.41 127 0)
 			(hide yes)
@@
 			)
 		)
-		(property "Value" "CL10A105KB8NNNC"
+		(property "Value" "1uF"
 			(at 114.3 92.71 0)
 			(hide yes)
@@
 			)
 		)
-		(property "Footprint" "easyeda2kicad:C0603"
+		(property "Footprint" "Capacitor_SMD:C_0603_1608Metric"
 			(at 114.3 104.14 0)
 			(hide yes)
@@
 			)
 		)
-		(property "Datasheet" "https://lcsc.com/product-detail/Multilayer-Ceramic-Capacitors-MLCC-SMD-SMT_SAMSUNG_CL10A105KB8NNNC_1uF-105-10-50V_C15849.html"
+		(property "Datasheet" ""
 			(at 114.3 106.68 0)
 			(hide yes)
@@
 			)
 		)
-		(property "Value" "CL10A105KB8NNNC"
+		(property "Value" "1uF"
 			(at 107.95 99.06 0)
 			(hide yes)
@@
 			)
 		)
-		(property "Footprint" "easyeda2kicad:C0603"
+		(property "Footprint" "Capacitor_SMD:C_0603_1608Metric"
 			(at 107.95 110.49 0)
 			(hide yes)
@@
 			)
 		)
-		(property "Datasheet" "https://lcsc.com/product-detail/Multilayer-Ceramic-Capacitors-MLCC-SMD-SMT_SAMSUNG_CL10A105KB8NNNC_1uF-105-10-50V_C15849.html"
+		(property "Datasheet" ""
 			(at 107.95 113.03 0)
 			(hide yes)
@@
 			)
 		)
-		(property "Footprint" "easyeda2kicad:C0805"
+		(property "Footprint" "Capacitor_SMD:C_0805_2012Metric"
 			(at 99.06 73.66 0)
 			(hide yes)
@@
 			)
 		)
-		(property "Datasheet" "https://lcsc.com/product-detail/Multilayer-Ceramic-Capacitors-MLCC-SMD-SMT_SAMSUNG_CL21A475KAQNNNE_4-7uF-475-10-25V_C1779.html"
+		(property "Datasheet" ""
 			(at 101.6 73.66 0)
 			(hide yes)
@@
 			)
 		)
-		(property "Value" "CL10A105KB8NNNC"
+		(property "Value" "1uF"
 			(at 123.19 102.87 0)
 			(hide yes)
@@
 			)
 		)
-		(property "Footprint" "easyeda2kicad:C0603"
+		(property "Footprint" "Capacitor_SMD:C_0603_1608Metric"
 			(at 123.19 114.3 0)
 			(hide yes)
@@
 			)
 		)
-		(property "Datasheet" "https://lcsc.com/product-detail/Multilayer-Ceramic-Capacitors-MLCC-SMD-SMT_SAMSUNG_CL10A105KB8NNNC_1uF-105-10-50V_C15849.html"
+		(property "Datasheet" ""
 			(at 123.19 116.84 0)
 			(hide yes)
@@
 			)
 		)
-		(property "Footprint" "easyeda2kicad:C0805"
+		(property "Footprint" "Capacitor_SMD:C_0805_2012Metric"
 			(at 50.8 73.66 0)
 			(hide yes)
@@
 			)
 		)
-		(property "Datasheet" "https://lcsc.com/product-detail/Multilayer-Ceramic-Capacitors-MLCC-SMD-SMT_SAMSUNG_CL21A475KAQNNNE_4-7uF-475-10-25V_C1779.html"
+		(property "Datasheet" ""
 			(at 53.34 73.66 0)
 			(hide yes)
@@
 			)
 		)
-		(property "Value" "0402WGF1002TCE"
+		(property "Value" "10k"
 			(at 116.8399 80.01 90)
 			(hide yes)
@@
 			)
 		)
-		(property "Datasheet" "https://lcsc.com/product-detail/Chip-Resistor-Surface-Mount-UniOhm_10KR-1002-1_C25744.html"
+		(property "Datasheet" ""
 			(at 115.57 72.39 0)
 			(hide yes)
@@
 			)
 		)
-		(property "Value" "0603WAF100KT5E"
+		(property "Value" "1"
 			(at 83.82 109.2199 90)
 			(hide yes)
@@
 			)
 		)
-		(property "Datasheet" "https://lcsc.com/product-detail/Chip-Resistor-Surface-Mount-UniOhm_1R-1R00-1_C22936.html"
+		(property "Datasheet" ""
 			(at 91.44 107.95 0)
 			(hide yes)
@@
 			)
 		)
-		(property "Value" "CL10A105KB8NNNC"
+		(property "Value" "1uF"
 			(at 120.65 118.11 0)
 			(hide yes)
@@
 			)
 		)
-		(property "Footprint" "easyeda2kicad:C0603"
+		(property "Footprint" "Capacitor_SMD:C_0603_1608Metric"
 			(at 120.65 129.54 0)
 			(hide yes)
@@
 			)
 		)
-		(property "Datasheet" "https://lcsc.com/product-detail/Multilayer-Ceramic-Capacitors-MLCC-SMD-SMT_SAMSUNG_CL10A105KB8NNNC_1uF-105-10-50V_C15849.html"
+		(property "Datasheet" ""
 			(at 120.65 132.08 0)
 			(hide yes)
@@
 			)
 		)
-		(property "Value" "0603WAF220KT5E"
+		(property "Value" "2.2"
 			(at 118.1099 76.2 90)
 			(hide yes)
@@
 			)
 		)
-		(property "Footprint" "easyeda2kicad:R0603"
+		(property "Footprint" "Resistor_SMD:R_0603_1608Metric"
 			(at 116.84 71.12 0)
 			(hide yes)
@@
 			)
 		)
-		(property "Datasheet" "https://lcsc.com/product-detail/Chip-Resistor-Surface-Mount-UniOhm_2-2R-2R20-1_C22939.html"
+		(property "Datasheet" ""
 			(at 116.84 68.58 0)
 			(hide yes)
@@
 			)
 		)
-		(property "Footprint" "easyeda2kicad:C0805"
+		(property "Footprint" "Capacitor_SMD:C_0805_2012Metric"
 			(at 123.19 60.96 0)
 			(hide yes)
@@
 			)
 		)
-		(property "Datasheet" "https://lcsc.com/product-detail/Multilayer-Ceramic-Capacitors-MLCC-SMD-SMT_SAMSUNG_CL21A475KAQNNNE_4-7uF-475-10-25V_C1779.html"
+		(property "Datasheet" ""
 			(at 123.19 58.42 0)
 			(hide yes)
@@
 			)
 		)
-		(property "Footprint" "easyeda2kicad:C0805"
+		(property "Footprint" "Capacitor_SMD:C_0805_2012Metric"
 			(at 107.95 121.92 0)
 			(hide yes)
@@
 			)
 		)
-		(property "Datasheet" "https://lcsc.com/product-detail/Multilayer-Ceramic-Capacitors-MLCC-SMD-SMT_SAMSUNG_CL21A475KAQNNNE_4-7uF-475-10-25V_C1779.html"
+		(property "Datasheet" ""
 			(at 107.95 124.46 0)
 			(hide yes)
